File: lots-of-serial.kicad_pcb (KiCad board)
At the start: 6 copper layers, 49.2 x 37.8 mm, 59 parts, among them J1 Conn_01x04, J2 Conn_01x04, J3 Conn_01x04, J4 Conn_01x04, J5 Conn_01x04, J6 Conn_01x04, J7 Conn_01x04, J8 Conn_01x04, SW1 SW_SPDT, SW2 SW_SPDT, SW3 SW_SPDT, SW4 SW_SPDT, U1 FE1.1s, U6 MAX232, U7 MAX232, Y1 12M

Commit message: Commit message. Stuff has happened. Not sure what. I think it's the middle of board version 3.0 now
Parts:
- moved D1 88.0 mm to (43.7, 90.9), turned to 180 degrees
- moved D2 87.8 mm to (43.7, 91.9)
- moved D3 87.5 mm to (43.7, 93.0), turned to 180 degrees
- moved D4 87.3 mm to (43.7, 94.0)
- moved D5 86.3 mm to (43.7, 89.9), turned to 180 degrees
- moved R1 76.4 mm to (44.2, 77.0), turned to 180 degrees
- moved R6 74.3 mm to (45.7, 89.9)
- moved R5 73.5 mm to (45.7, 93.0), turned to 180 degrees
- moved R4 73.5 mm to (45.7, 91.4), turned to 180 degrees
- moved R2 72.6 mm to (47.0, 84.6), turned to 90 degrees
- moved C6 67.5 mm to (54.6, 65.3)
- moved Y1 67.2 mm to (58.4, 86.4), turned to -90 degrees
- moved C5 65.4 mm to (47.8, 82.0), turned to -90 degrees
- moved C7 65.3 mm to (54.6, 71.4)
- moved R3 65.2 mm to (56.4, 78.7), turned to 180 degrees
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Routing:
- net VBUS: track 0.00 -> 98.8 mm, vias 0 -> 4
- net +3V3: track 0.00 -> 62.3 mm, vias 0 -> 6
- net Vo2: track 0.00 -> 38.3 mm, vias 0 -> 1
- net Vo3: track 0.00 -> 37.4 mm
- net Vo1: track 0.00 -> 35.4 mm, vias 0 -> 2
- net Vo4: track 0.00 -> 35.1 mm, vias 0 -> 2
- net Net-(D1-A): track 0.00 -> 14.5 mm, vias 0 -> 2
- net TX1: track 0.00 -> 13.8 mm
- net 232_TX2: track 0.00 -> 12.5 mm, vias 0 -> 1
- net 232_RX2: track 0.00 -> 12.5 mm, vias 0 -> 1
- net 232_RX4: track 0.00 -> 12.5 mm, vias 0 -> 1
- net 232_TX4: track 0.00 -> 12.5 mm, vias 0 -> 1
- net +1V8: track 0.00 -> 12.1 mm
- net TX2: track 0.00 -> 11.6 mm, vias 0 -> 1
- net RX2: track 0.00 -> 11.4 mm, vias 0 -> 2
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- added copper zone on F.Cu, net GND
Other:
- board size 49.2 x 37.8 mm -> 41.4 x 37.8 mm
- board text added: "1"
- board text added: "2"
- board text added: "3"
- board text added: "4"
- board text added: "GND"
- board text added: "RX"
- board text added: "TX"
- board text added: "VCC"

Commit message: Likely acceptable version 2
Routing:
- net VBUS: track 98.8 -> 98.1 mm
- net GND: vias 3 -> 5
Changed lines of the file:
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@@
     )
   )
-  (gr_rect (start 47.498 80.772) (end 48.26 81.788)
-    (stroke (width 0.11) (type solid)) (fill solid) (layer "F.Cu"))
   (gr_rect (start 36.9824 64.1604) (end 78.4098 101.9556)
     (stroke (width 0.05) (type default)) (fill none) (layer "Edge.Cuts"))
@@
   (segment (start 69.695 68.834) (end 69.342 68.834) (width 0.3) (layer "F.Cu") (net 2))
   (via (at 47.498 83.058) (size 0.6) (drill 0.25) (layers "F.Cu" "B.Cu") (free) (net 2))
+  (via (at 42.926 88.392) (size 0.6) (drill 0.25) (layers "F.Cu" "B.Cu") (free) (net 2))
   (via (at 43.942 84.074) (size 0.6) (drill 0.25) (layers "F.Cu" "B.Cu") (free) (net 2))
   (via (at 50.165 81.534) (size 0.6) (drill 0.25) (layers "F.Cu" "B.Cu") (net 2))
+  (via (at 46.736 78.613) (size 0.6) (drill 0.25) (layers "F.Cu" "B.Cu") (free) (net 2))
   (segment (start 48.501 84.6455) (end 49.216 84.6455) (width 0.15) (layer "F.Cu") (net 3))
   (segment (start 46.736 92.964) (end 46.738 92.962) (width 0.15) (layer "F.Cu") (net 3))
@@
   (segment (start 45.193 80.608) (end 44.36 80.608) (width 0.25) (layer "F.Cu") (net 24))
   (segment (start 40.546 70.902) (end 42.164 70.866) (width 0.25) (layer "F.Cu") (net 24))
+  (segment (start 47.752 80.8355) (end 49.216 80.8355) (width 0.25) (layer "F.Cu") (net 24))
   (segment (start 63.311 99.187) (end 64.389 99.187) (width 0.25) (layer "F.Cu") (net 24))
-  (segment (start 48.366 80.8355) (end 49.216 80.8355) (width 0.25) (layer "F.Cu") (net 24))
+  (segment (start 46.3955 80.8355) (end 47.752 80.8355) (width 0.25) (layer "F.Cu") (net 24))
   (segment (start 43.18 84.582) (end 42.164 85.598) (width 0.25) (layer "F.Cu") (net 24))
   (segment (start 45.193 80.608) (end 46.168 80.608) (width 0.25) (layer "F.Cu") (net 24))
@@
   (segment (start 42.164 85.598) (end 42.164 90.678) (width 0.25) (layer "F.Cu") (net 24))
   (segment (start 43.965994 85.09) (end 44.383994 85.508) (width 0.25) (layer "F.Cu") (net 24))
+  (segment (start 49.216 82.1055) (end 48.2955 82.1055) (width 0.2) (layer "F.Cu") (net 24))
   (segment (start 42.164 97.412) (end 41.184 98.392) (width 0.25) (layer "F.Cu") (net 24))
-  (segment (start 48.26 81.9995) (end 48.26 80.9415) (width 0.25) (layer "F.Cu") (net 24))
   (segment (start 47.117 77.724) (end 61.242 77.724) (width 0.25) (layer "F.Cu") (net 24))
   (segment (start 42.164 75.184) (end 42.164 80.518) (width 0.25) (layer "F.Cu") (net 24))
+  (segment (start 48.2955 82.1055) (end 47.752 81.562) (width 0.2) (layer "F.Cu") (net 24))
   (segment (start 42.164 70.866) (end 42.128 70.902) (width 0.25) (layer "F.Cu") (net 24))
   (segment (start 63.311 100.42) (end 63.274 100.457) (width 0.25) (layer "F.Cu") (net 24))
@@
   (segment (start 43.18 81.534) (end 43.18 84.582) (width 0.25) (layer "F.Cu") (net 24))
   (segment (start 63.311 99.187) (end 63.311 100.42) (width 0.25) (layer "F.Cu") (net 24))
-  (segment (start 46.3955 80.8355) (end 49.216 80.8355) (width 0.25) (layer "F.Cu") (net 24))
   (segment (start 43.688 85.09) (end 43.965994 85.09) (width 0.25) (layer "F.Cu") (net 24))
-  (segment (start 48.26 80.9415) (end 48.366 80.8355) (width 0.25) (layer "F.Cu") (net 24))
-  (segment (start 49.216 82.1055) (end 48.366 82.1055) (width 0.25) (layer "F.Cu") (net 24))
   (segment (start 42.164 70.866) (end 42.926 70.866) (width 0.25) (layer "F.Cu") (net 24))
-  (segment (start 48.366 82.1055) (end 48.26 81.9995) (width 0.25) (layer "F.Cu") (net 24))
   (segment (start 65.278 98.298) (end 65.278 81.76) (width 0.25) (layer "F.Cu") (net 24))
   (segment (start 64.389 99.187) (end 65.278 98.298) (width 0.25) (layer "F.Cu") (net 24))
+  (segment (start 47.752 81.562) (end 47.752 80.8355) (width 0.2) (layer "F.Cu") (net 24))
   (segment (start 43.688 81.026) (end 43.18 81.534) (width 0.25) (layer "F.Cu") (net 24))
   (via (at 42.164 70.866) (size 0.6) (drill 0.25) (layers "F.Cu" "B.Cu") (net 24))
